Commit message: feat(interface): ee_twist on ArmState; make the URDF mesh paths portable
Two things a ROS frontend needs and could not get.

**ee_twist.** The pump already computes ee_pose with fk(q) every tick and hands it out
on ArmState. A client doing anything Cartesian -- and after Plan 2 most of the streaming
controllers are -- had the tool's pose but not its velocity, and no way to get one that
agreed with the pose. So the pump now also runs jacobian(q) and stores J*qd beside it.

Same model, same feedback sample, so the two agree by construction. It is
LOCAL_WORLD_ALIGNED, matching Dynamics::jacobian: a world-aligned frame at the tool, not
the body frame. Deliberately NOT read from the arm's own tool_twist feedback -- that is a
different frame and a different model from the ee_pose beside it, and the two would
silently disagree by the arm's configured tool offset. The Jacobian is preallocated; the
pump is not an RT thread but allocating a 6x7 every 10 ms for no reason is not what this
repo does.

The test computes J*qd independently rather than re-reading what the pump wrote, so a
regression shows up as a mismatch instead of a plausible-looking wrong number.

**The URDF mesh paths.** All 37 pointed at absolute paths inside a container that no
longer exists:

    file:///root/c3pzero_ws/install/kortex_description/share/kortex_description/...

which resolves nowhere. Pinocchio never noticed because buildModel ignores geometry, so
the driver was fine -- but the URDF was unloadable by anything that does read meshes:
RViz, any description package, any real2sim work. Rewritten to package:// against the
three packages actually referenced (kortex_description, realsense2_description,
robotiq_description), plus a stray meshes// double slash.

Co-Authored-By: Claude Opus 5 (1M context) <noreply@anthropic.com>
Claude-Session: https://claude.ai/code/session_01RXbb4Ew5jSLgeT8W33tjLt

File: models/gen3_7dof_2f85.urdf (robot description, URDF)
Before this commit: robot gen3_, 31 links, 30 joints
Links:
- link gen3_base_link: geometry collision mesh filename=package://kortex_description/arms/gen3/7dof/meshes/base_lin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; visual mesh filename=package://kortex_description/arms/gen3/7dof/meshes/base_lin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
- link gen3_bracelet_link: geometry collision mesh filename=package://kortex_description/arms/gen3/7dof/meshes/bracelet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; visual mesh filename=package://kortex_description/arms/gen3/7dof/meshes/bracelet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
- link gen3_forearm_link: geometry collision mesh filename=package://kortex_description/arms/gen3/7dof/meshes/forearm_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; visual mesh filename=package://kortex_description/arms/gen3/7dof/meshes/forearm_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
- link gen3_half_arm_1_link: geometry collision mesh filename=package://kortex_description/arms/gen3/7dof/meshes/half_arm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; visual mesh filename=package://kortex_description/arms/gen3/7dof/meshes/half_arm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
- link gen3_half_arm_2_link: geometry collision mesh filename=package://kortex_description/arms/gen3/7dof/meshes/half_arm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; visual mesh filename=package://kortex_description/arms/gen3/7dof/meshes/half_arm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
- link gen3_robotiq_85_base_link: geometry collision mesh filename=package://robotiq_description/meshes/collision/robotiq_base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; visual mesh filename=package://robotiq_description/meshes/visual/robotiq_base.dae
- link gen3_robotiq_85_left_finger_link: geometry collision mesh filename=package://robotiq_description/meshes/collision/left_finger.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; visual mesh filename=package://robotiq_description/meshes/visual/left_finger.dae
- link gen3_robotiq_85_left_finger_tip_link: geometry collision mesh filename=package://robotiq_description/meshes/collision/left_finger_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; visual mesh filename=package://robotiq_description/meshes/visual/left_finger_tip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
- link gen3_robotiq_85_left_inner_knuckle_link: geometry collision mesh filename=package://robotiq_description/meshes/collision/left_inner_k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; visual mesh filename=package://robotiq_description/meshes/visual/left_inner_knuc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
- link gen3_robotiq_85_left_knuckle_link: geometry collision mesh filename=package://robotiq_description/meshes/collision/left_knuckle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; visual mesh filename=package://robotiq_description/meshes/visual/left_knuckle.dae
- link gen3_robotiq_85_right_finger_link: geometry collision mesh filename=package://robotiq_description/meshes/collision/right_finger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; visual mesh filename=package://robotiq_description/meshes/visual/right_finger.dae
- link gen3_robotiq_85_right_finger_tip_link: geometry collision mesh filename=package://robotiq_description/meshes/collision/right_finger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; visual mesh filename=package://robotiq_description/meshes/visual/right_finger_ti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
- link gen3_robotiq_85_right_inner_knuckle_link: geometry collision mesh filename=package://robotiq_description/meshes/collision/right_inner_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; visual mesh filename=package://robotiq_description/meshes/visual/right_inner_knu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
- link gen3_robotiq_85_right_knuckle_link: geometry collision mesh filename=package://robotiq_description/meshes/collision/right_knuckl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; visual mesh filename=package://robotiq_description/meshes/visual/right_knuckle.d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
- link gen3_shoulder_link: geometry collision mesh filename=package://kortex_description/arms/gen3/7dof/meshes/shoulder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; visual mesh filename=package://kortex_description/arms/gen3/7dof/meshes/shoulder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
- link gen3_spherical_wrist_1_link: geometry collision mesh filename=package://kortex_description/arms/gen3/7dof/meshes/spherica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; visual mesh filename=package://kortex_description/arms/gen3/7dof/meshes/spherica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
- link gen3_spherical_wrist_2_link: geometry collision mesh filename=package://kortex_description/arms/gen3/7dof/meshes/spherica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; visual mesh filename=package://kortex_description/arms/gen3/7dof/meshes/spherica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
- link wrist_camera_mount_link: geometry collision mesh filename=package://kortex_description/arms/gen3/7dof/meshes/realsens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; visual mesh filename=package://kortex_description/arms/gen3/7dof/meshes/realsens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
- link wrist_mounted_camera_link: geometry collision box size=0.02005 0.099 0.023; visual mesh filename=package://realsense2_description/meshes/d415.stl
